File: fever-hat.sch (KiCad schematic (older format))
At the start: 36 parts, among them IC1 MPM3630GQV-P, IC2 TPS2540RTET, J1 Raspberry_Pi_2_3, J2 Thermal Camera, J3 USB_B, J4 USB_A, J5 Conn_01x04, J6 Barrel_Jack_Switch, Q1 Q_NMOS_GSD, Q2 Q_PMOS_DGS

Commit message: Smaller PCB and use buck converter that JLCPCB can provide
Parts:
- removed C1, C2, C3, C8: 22uF, Capacitor_SMD:C_0805_2012Metric, symbol Device:C
- removed IC1: MPM3630GQV-P, MPM3630GQV-P:QFN-20(3MMX5MMX1.6MM), symbol MPM3630GQV-P:MPM3630GQV-P
- removed IC2: TPS2540RTET, TPS2540RTET:QFN50P300X300X80-17N-D, symbol TPS2540RTET:TPS2540RTET
- removed R4: 100K, Resistor_SMD:R_0603_1608Metric, symbol Device:R
- removed RV1: R_POT_TRIM, Potentiometer_SMD:Potentiometer_Bourns_TC33X_Vertical, symbol Device:R_POT_TRIM
- added C10: 220uF, Capacitor_SMD:CP_Elec_6.3x7.7, symbol Device:CP1
- added C4: 10uF, Capacitor_SMD:C_0805_2012Metric, symbol Device:C
- added C9: 0.01uF, Capacitor_SMD:C_0603_1608Metric, symbol Device:C
- added D1: B340A, Diode_SMD:D_SMA, symbol Device:D_Shockley
- added D2: D_Zener, Diode_SMD:D_SMA, symbol Device:D_Zener
- added D3: LED, Diode_SMD:D_0603_1608Metric, symbol Device:LED
- added IC1: TPS2546RTER, QFN50P300X300X80-17N-D, symbol TPS2546RTER:TPS2546RTER
- added L1: 15uH, Inductor_SMD:L_10.4x10.4_H4.8, symbol pspice:INDUCTOR
- added R12: 3K16, Resistor_SMD:R_0603_1608Metric, symbol Device:R
- added R6: 10K, Resistor_SMD:R_0603_1608Metric, symbol Device:R
- added U1: TPS5430DDA, Package_SO:TI_SO-PowerPAD-8_ThermalVias, symbol Regulator_Switching:TPS5430DDA
- C5, C7: LCSC Part # (none) -> C45783
- C6: LCSC Part # (none) -> C15849
- F1: LCSC Part # (none) -> C182718
- FID1, FID2, FID3, H1, H2, H3, H4: Skip BOM (none) -> True
- Q1: LCSC Part # (none) -> C20917
- Q2: value Q_PMOS_DGS -> Q_PMOS_GDS; footprint footprints:IRF9310PbF -> Package_TO_SOT_SMD:SOT-23; symbol Device:Q_PMOS_DGS -> Device:Q_PMOS_GSD; LCSC Part # (none) -> C15127
- R1, R10, R11, R8, R9: LCSC Part # (none) -> C25803
- R2: value 51K -> 100K; DigiKeyPN RMCF0603FT51K0CT-ND -> RR08P100KDCT-ND; LCSC Part # (none) -> C25803
- R3: value 6K98 -> 470R; DigiKeyPN P20069CT-ND -> 311-470HRCT-ND; LCSC Part # (none) -> C23179
- R5: LCSC Part # (none) -> C23179
- R7: value 39K -> 36K; LCSC Part # (none) -> C23147
Connections:
- net +5V: now also C10.1, IC1.1 (IN), IC1.4 (ILIM_SEL), L1.2, R6.1
- net D_IN_N: now also IC1.11 (DM_IN)
- net D_IN_P: now also IC1.10 (DP_IN)
- net D_OUT_N: now also IC1.2 (DM_OUT)
- net D_OUT_P: now also IC1.3 (DP_OUT)
- net GND: now also R2.2, C10.2, C4.2, D1.2 (A), D3.1 (K), IC1.14 (GND), IC1.17 (EP_GND), R12.2, U1.6 (GND), U1.9 (GNDPAD); no longer Q2.2 (G), R3.2
- net LED_INDICATOR: now also R3.1
- net RESET: now also U1.5 (EN)
- net VCC: now also C7.1, Q2.2 (S), C4.1, D2.1 (K), U1.7 (VIN); no longer F1.1
- net at C5.1, J4.1 (VBUS): now also IC1.12 (OUT)
- net at R2.1: now also Q2.1 (G), D2.2 (A)
- net at R7.2: now also IC1.16 (ILIM_HI)
- net at R11.2: now also IC1.5 (EN)
- net at R10.2: now also IC1.6 (CLT1)
- net at R9.2: now also IC1.7 (CLT2)
- net at R8.2: now also IC1.8 (CLT3)
- net at J6.1: now also F1.2; no longer Q2.1 (D)
- new net: C9.2, U1.1 (BOOT)
- new net: R12.1, R6.2, U1.4 (VSENSE)
- new net: C9.1, D1.1 (K), L1.1, U1.8 (PH)
- new net: D3.2 (A), R3.2
- new net: F1.1, Q2.3 (D)
- no-connect marks 31 -> 26
Other:
- moved on the sheet: C5, C6, C7, F1, FID1, FID2, FID3, H1, H2, H3, H4, J3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

Commit message: Update unductor footprint
Parts:
- removed J3: USB_B, Connector_USB:USB_B_Lumberg_2411_02_Horizontal, symbol Connector:USB_B
- added J3: Conn_01x02, Connector_JST:JST_PH_S2B-PH-K_1x02_P2.00mm_Horizontal, symbol Connector_Generic:Conn_01x02
- J5: footprint Connector_JST:JST_PH_B4B-PH-K_1x04_P2.00mm_Vertical -> Connector_JST:JST_PH_S4B-PH-K_1x04_P2.00mm_Horizontal
- L1: footprint Inductor_SMD:L_10.4x10.4_H4.8 -> footprints:MWSA1004-150MT
Connections:
- net D_OUT_N: now also J3.1 (Pin_1)
- net D_OUT_P: now also J3.2 (Pin_2)
- no-connect marks 26 -> 25
Changed lines of the file:
@@
 F 0 "J5" H 8218 625 50  0000 C CNN
 F 1 "Conn_01x04" H 8218 716 50  0000 C CNN
-F 2 "Connector_JST:JST_PH_B4B-PH-K_1x04_P2.00mm_Vertical" H 8300 1050 50  0001 C CNN
+F 2 "Connector_JST:JST_PH_S4B-PH-K_1x04_P2.00mm_Horizontal" H 8300 1050 50  0001 C CNN
 F 3 "~" H 8300 1050 50  0001 C CNN
 F 4 "455-1706-ND" H 8300 1050 50  0001 C CNN "DigiKeyPN"
@@
 F 0 "L1" H 3500 3365 50  0000 C CNN
 F 1 "15uH" H 3500 3274 50  0000 C CNN
-F 2 "Inductor_SMD:L_10.4x10.4_H4.8" H 3500 3150 50  0001 C CNN
+F 2 "footprints:MWSA1004-150MT" H 3500 3150 50  0001 C CNN
 F 3 "~" H 3500 3150 50  0001 C CNN
 F 4 "C151872" H 3500 3150 50  0001 C CNN "LCSC Part #"
@@
 $EndComp
 Wire Wire Line
-	6200 5050 6200 5000
-$Comp
-L power:GND #PWR0116
-U 1 1 5F2D495D
-P 6150 5100
-F 0 "#PWR0116" H 6150 4850 50  0001 C CNN
-F 1 "GND" H 6155 4927 50  0000 C CNN
-F 2 "" H 6150 5100 50  0001 C CNN
-F 3 "" H 6150 5100 50  0001 C CNN
-	1    6150 5100
-	1    0    0    -1
-$EndComp
-NoConn ~ 6500 4400
-Wire Wire Line
 	6900 4650 6900 4600
 Wire Wire Line
@@
 Wire Wire Line
 	7300 4600 7050 4600
-$Comp
-L Connector:USB_B J3
-U 1 1 5F07EC5A
-P 6200 4600
-F 0 "J3" H 6257 5067 50  0000 C CNN
-F 1 "USB_B" H 6257 4976 50  0000 C CNN
-F 2 "Connector_USB:USB_B_Lumberg_2411_02_Horizontal" H 6350 4550 50  0001 C CNN
-F 3 " ~" H 6350 4550 50  0001 C CNN
-F 4 "ED2983-ND" H 6200 4600 50  0001 C CNN "DigiKeyPN"
-	1    6200 4600
-	1    0    0    -1
-$EndComp
 Wire Wire Line
 	7300 4700 7250 4700
@@
 Wire Wire Line
 	8950 4600 8950 4650
-Wire Wire Line
-	6100 5000 6100 5050
-Wire Wire Line
-	6100 5050 6150 5050
-Wire Wire Line
-	6150 5100 6150 5050
-Connection ~ 6150 5050
-Wire Wire Line
-	6150 5050 6200 5050
 Wire Wire Line
 	7150 4800 7150 4500
@@
 	8150 1850 8150 1900
 $Comp
-L power:PWR_FLAG #FLG?
+L power:PWR_FLAG #FLG0101
 U 1 1 5F2ECABA
 P 4550 3100
-F 0 "#FLG?" H 4550 3175 50  0001 C CNN
+F 0 "#FLG0101" H 4550 3175 50  0001 C CNN
 F 1 "PWR_FLAG" H 4550 3273 50  0000 C CNN
 F 2 "" H 4550 3100 50  0001 C CNN
@@
 	4550 3150 4550 3100
 Connection ~ 4350 3150
+$Comp
+L Connector_Generic:Conn_01x02 J3
+U 1 1 5F30BA68
+P 6300 4700
+F 0 "J3" H 6500 4400 50  0000 C CNN
+F 1 "Conn_01x02" H 6450 4500 50  0000 C CNN
+F 2 "Connector_JST:JST_PH_S2B-PH-K_1x02_P2.00mm_Horizontal" H 6300 4700 50  0001 C CNN
+F 3 "~" H 6300 4700 50  0001 C CNN
+	1    6300 4700
+	-1   0    0    1
+$EndComp
 $EndSCHEMATC
